Commit message: error gone? :D

File: install/udm_pioneer_p3dx/share/udm_pioneer_p3dx/urdf/pioneer3dx.gazebo.xacro (robot description, xacro)
@@ -16,5 +16,5 @@
 <robot name="pioneer_gazebo" xmlns:xacro="http://ros.org/wiki/xacro">
   <!-- properties (constants) -->
-  <property name="ns" value="p3dx" />
+  <xacro:property name="ns" value="p3dx" />
   <!-- base_link -->
 	<gazebo reference="base_link">
@@ -105,7 +105,4 @@
 				<noise>
 					<type>gaussian</type>
-					<!-- Noise parameters based on published spec for Hokuyo laser achieving
-						"+-30mm" accuracy at range < 10m. A mean of 0.0m and stddev of 0.01m will
-						put 99.7% of samples within 0.03m of the true reading. -->
 					<mean>0.0</mean>
 					<stddev>0.01</stddev>

File: install/udm_pioneer_p3dx/share/udm_pioneer_p3dx/urdf/pioneer3dx.xacro (robot description, xacro)
@@ -3,8 +3,4 @@
 This is the xacro description of a Pioneer 3DX, to be used in rviz and gazebo.
 Copyright (C) 2013 Rafael Berkvens rafael.berkvens@uantwerpen.be
-This program is free software: you can redistribute it and/or modify
-it under the terms of the GNU General Public License as published by
-the Free Software Foundation, either version 3 of the License, or
-(at your option) any later version.
 This program is distributed in the hope that it will be useful,
 but WITHOUT ANY WARRANTY; without even the implied warranty of
@@ -18,7 +14,7 @@
 <robot name="pioneer3dx" xmlns:xacro="http://ros.org/wiki/xacro">
   <!-- import all gazebo-customization elements, including gazebo colors -->
-  <xacro:include filename="$(find p3dx_description)/urdf/pioneer3dx.gazebo.xacro" />
+  <xacro:include filename="$(find udm_pioneer_p3dx)/urdf/pioneer3dx.gazebo.xacro" />
   <!-- import the pioneer 3dx's wheels -->
-  <xacro:include filename="$(find p3dx_description)/urdf/pioneer3dx_wheel.xacro" />
+  <xacro:include filename="$(find udm_pioneer_p3dx)/urdf/pioneer3dx_wheel.xacro" />
   <!-- chassis -->
 	<link name="base_link">

File: install/udm_pioneer_p3dx/share/udm_pioneer_p3dx/urdf/pioneer3dx_1.gazebo.xacro (robot description, xacro)
@@ -16,5 +16,5 @@
 <robot name="pioneer_gazebo" xmlns:xacro="http://ros.org/wiki/xacro">
   <!-- properties (constants) -->
-  <property name="ns" value="p3dx" />
+  <xacro:property name="ns" value="p3dx" />
   <!-- base_link -->
 	<gazebo reference="base_link">

File: install/udm_pioneer_p3dx/share/udm_pioneer_p3dx/urdf/pioneer3dx_wheel.xacro (robot description, xacro)
@@ -18,5 +18,5 @@
 <robot xmlns:xacro="http://ros.org/wiki/xacro">
 	<!-- properties (constants) -->
-	<property name="M_PI" value="3.14159" />
+	<xacro:property name="M_PI" value="3.14159" />
 	<!-- right/left hubcap + wheel -->
 	<xacro:macro name="p3dx_wheel" params="suffix parent reflect">

Commit message: Working on making the colors show

File: install/udm_pioneer_p3dx/share/udm_pioneer_p3dx/urdf/pioneer3dx.gazebo.xacro (robot description, xacro)
@@ -19,21 +19,21 @@
   <!-- base_link -->
 	<gazebo reference="base_link">
-		<material>Gazebo/Red</material>
+		<material value="Gazebo/Red" />
 	</gazebo>
   <!-- top_plate -->
   <gazebo reference="top_plate">
-    <material>Gazebo/Black</material>
+    <material value="Gazebo/Red" />
   </gazebo>
   <!-- swivel -->
   <gazebo reference="swivel">
-    <material>Gazebo/Grey</material>
+    <material value="Gazebo/Grey" />
   </gazebo>
   <!-- center_hubcap -->
 	<gazebo reference="center_hubcap">
-		<material>Gazebo/Grey</material>
+		<material value="Gazebo/Grey">Gazebo/Grey</material>
 	</gazebo>
   <!-- center_wheel -->
 	<gazebo reference="center_wheel">
-		<material>Gazebo/Black</material>
+		<material value="Gazebo/Black">Gazebo/Black</material>
 		<mu1>10.0</mu1>
 		<mu2>10.0</mu2>

File: install/udm_pioneer_p3dx/share/udm_pioneer_p3dx/urdf/pioneer3dx.xacro (robot description, xacro)
@@ -53,5 +53,5 @@
 				<mesh filename="package://udm_pioneer_p3dx/p3dx_description/meshes/top.stl" />
 			</geometry>
-			<material name="TopBlack">
+			<material>
 				<color rgba="0.038 0.038 0.038 1.0" />
 			</material>
@@ -200,5 +200,5 @@
 			<inertia ixx="1e-6" ixy="0" ixz="0" iyy="1e-6" iyz="0" izz="1e-6" />
 		</inertial>
-		<visual>
+		<visual name="lms_100">
 			<origin xyz="0 0 0" rpy="0 0 0" />
 			<geometry>

File: install/udm_pioneer_p3dx/share/udm_pioneer_p3dx/urdf/pioneer3dx_wheel.xacro (robot description, xacro)
@@ -29,5 +29,5 @@
 					iyz="0" izz="0.011763977943" />
 			</inertial>
-			<visual>
+			<visual name="p3dx_${suffix}_wheel_vis">
 				<origin xyz="0 0 0" rpy="0 0 0" />
 				<geometry name="pioneer_geom">
@@ -59,5 +59,5 @@
 					iyz="0" izz="0.011763977943" />
 			</inertial>
-			<visual>
+			<visual name="p3dx_${suffix}_hubcap_vis">
 				<origin xyz="0 0 0" rpy="0 0 0" />
 				<geometry name="pioneer_geom">

Commit message: fixing bug

File: install/udm_pioneer_p3dx/share/udm_pioneer_p3dx/urdf/pioneer3dx.gazebo.xacro (robot description, xacro)
@@ -18,30 +18,30 @@
   <xacro:property name="ns" value="p3dx" />
   <!-- base_link -->
-	<gazebo reference="base_link">
-		<material value="Gazebo/Red" />
-	</gazebo>
+  <gazebo reference="base_link">
+    <material>Gazebo/Red</material>
+  </gazebo>
   <!-- top_plate -->
   <gazebo reference="top_plate">
-    <material value="Gazebo/Red" />
+    <material>Gazebo/Red</material>
   </gazebo>
   <!-- swivel -->
   <gazebo reference="swivel">
-    <material value="Gazebo/Grey" />
+    <material>Gazebo/Grey</material>
   </gazebo>
   <!-- center_hubcap -->
-	<gazebo reference="center_hubcap">
-		<material value="Gazebo/Grey">Gazebo/Grey</material>
-	</gazebo>
+  <gazebo reference="center_hubcap">
+    <material>Gazebo/Grey</material>
+  </gazebo>
   <!-- center_wheel -->
-	<gazebo reference="center_wheel">
-		<material value="Gazebo/Black">Gazebo/Black</material>
-		<mu1>10.0</mu1>
-		<mu2>10.0</mu2>
-		<kp>1000000.0</kp>
-		<kd>1.0</kd>
-	</gazebo>
+  <gazebo reference="center_wheel">
+   <material>Gazebo/Black</material>
+    <mu1>10.0</mu1>
+    <mu2>10.0</mu2>
+    <kp>1000000.0</kp>
+    <kd>1.0</kd>
+  </gazebo>
   <!-- front_sonar -->
   <gazebo reference="front_sonar">
-    <material value="Gazebo/Yellow" />
+    <material>Gazebo/Yellow</material>
   </gazebo>
   <!-- differential drive -->
@@ -85,4 +85,5 @@
 	<!-- lms100 -->
 	<gazebo reference="lms100">
+		<material>Gazebo/Red</material>
 		<sensor type="ray" name="head_hokuyo_sensor">
 			<pose>0 0 0 0 0 0</pose>

File: install/udm_pioneer_p3dx/share/udm_pioneer_p3dx/urdf/pioneer3dx.xacro (robot description, xacro)
@@ -53,9 +53,9 @@
 				<mesh filename="package://udm_pioneer_p3dx/p3dx_description/meshes/top.stl" />
 			</geometry>
-			<material>
+			<material name="top_plate_material">
 				<color rgba="0.038 0.038 0.038 1.0" />
 			</material>
 		</visual>
-		<collision>
+		<collision name="top_plate_collision">
 			<origin xyz="0.0 0 0" rpy="0 0 0" />
 			<geometry name="pioneer_geom">
