Commit message: Updaing meshes

File: install/udm_pioneer_p3dx/share/udm_pioneer_p3dx/urdf/pioneer3dx.xacro (robot description, xacro)
@@ -28,5 +28,5 @@
 			<origin xyz="-0.045 0 0.148" rpy="0 0 0" />
 			<geometry name="pioneer_geom">
-				<mesh filename="package://p3dx_description/meshes/chassis.stl" />
+				<mesh filename="$(find udm_pioneer_p3dx)/p3dx_description/meshes/chassis.stl" />
 			</geometry>
 			<material name="ChassisRed">
@@ -51,5 +51,5 @@
 			<origin xyz="0 0 0" rpy="0 0 0" />
 			<geometry name="top_geom">
-				<mesh filename="package://p3dx_description/meshes/top.stl" />
+				<mesh filename="$(find udm_pioneer_p3dx)/p3dx_description/meshes/top.stl" />
 			</geometry>
 			<material name="TopBlack">
@@ -79,5 +79,5 @@
 			<origin xyz="0 0 0" rpy="0 0 0" />
 			<geometry name="pioneer_geom">
-				<mesh filename="package://p3dx_description/meshes/swivel.stl" />
+				<mesh filename="$(find udm_pioneer_p3dx)/p3dx_description/meshes/swivel.stl" />
 			</geometry>
 			<material name="swivel">
@@ -112,5 +112,5 @@
 			<origin xyz="0 0 0" rpy="0 0 0" />
 			<geometry name="pioneer_geom">
-				<mesh filename="package://p3dx_description/meshes/center_hubcap.stl" />
+				<mesh filename="$(find udm_pioneer_p3dx)/p3dx_description/meshes/center_hubcap.stl" />
 			</geometry>
 			<material name="swivel">
@@ -145,5 +145,5 @@
 			<origin xyz="0 0 0" rpy="0 0 0" />
 			<geometry name="pioneer_geom">
-				<mesh filename="package://p3dx_description/meshes/center_wheel.stl" />
+				<mesh filename="$(find udm_pioneer_p3dx)/p3dx_description/meshes/center_wheel.stl" />
 			</geometry>
 			<material name="WheelBlack">
@@ -175,5 +175,5 @@
 			<origin rpy="0 0 0" xyz="0 0 0" />
 			<geometry name="pioneer_geom">
-				<mesh filename="package://p3dx_description/meshes/front_sonar.stl" />
+				<mesh filename="$(find udm_pioneer_p3dx)/p3dx_description/meshes/front_sonar.stl" />
 			</geometry>
 			<material name="SonarYellow">
@@ -203,5 +203,5 @@
 			<origin xyz="0 0 0" rpy="0 0 0" />
 			<geometry>
-				<mesh filename="package://p3dx_description/meshes/lms100.dae" />
+				<mesh filename="$(find udm_pioneer_p3dx)/p3dx_description/meshes/lms100.dae" />
 			</geometry>
 		</visual>

Commit message: Getting robots showing, barely

File: install/udm_pioneer_p3dx/share/udm_pioneer_p3dx/urdf/pioneer3dx.xacro (robot description, xacro)
@@ -28,5 +28,5 @@
 			<origin xyz="-0.045 0 0.148" rpy="0 0 0" />
 			<geometry name="pioneer_geom">
-				<mesh filename="$(find udm_pioneer_p3dx)/p3dx_description/meshes/chassis.stl" />
+				<mesh filename="package://udm_pioneer_p3dx/p3dx_description/meshes/chassis.stl" />
 			</geometry>
 			<material name="ChassisRed">
@@ -51,5 +51,5 @@
 			<origin xyz="0 0 0" rpy="0 0 0" />
 			<geometry name="top_geom">
-				<mesh filename="$(find udm_pioneer_p3dx)/p3dx_description/meshes/top.stl" />
+				<mesh filename="package://udm_pioneer_p3dx/p3dx_description/meshes/top.stl" />
 			</geometry>
 			<material name="TopBlack">
@@ -79,5 +79,5 @@
 			<origin xyz="0 0 0" rpy="0 0 0" />
 			<geometry name="pioneer_geom">
-				<mesh filename="$(find udm_pioneer_p3dx)/p3dx_description/meshes/swivel.stl" />
+				<mesh filename="package://udm_pioneer_p3dx/p3dx_description/meshes/swivel.stl" />
 			</geometry>
 			<material name="swivel">
@@ -112,5 +112,5 @@
 			<origin xyz="0 0 0" rpy="0 0 0" />
 			<geometry name="pioneer_geom">
-				<mesh filename="$(find udm_pioneer_p3dx)/p3dx_description/meshes/center_hubcap.stl" />
+				<mesh filename="package://udm_pioneer_p3dx/p3dx_description/meshes/center_hubcap.stl" />
 			</geometry>
 			<material name="swivel">
@@ -145,5 +145,5 @@
 			<origin xyz="0 0 0" rpy="0 0 0" />
 			<geometry name="pioneer_geom">
-				<mesh filename="$(find udm_pioneer_p3dx)/p3dx_description/meshes/center_wheel.stl" />
+				<mesh filename="package://udm_pioneer_p3dx/p3dx_description/meshes/center_wheel.stl" />
 			</geometry>
 			<material name="WheelBlack">
@@ -175,5 +175,5 @@
 			<origin rpy="0 0 0" xyz="0 0 0" />
 			<geometry name="pioneer_geom">
-				<mesh filename="$(find udm_pioneer_p3dx)/p3dx_description/meshes/front_sonar.stl" />
+				<mesh filename="package://udm_pioneer_p3dx/p3dx_description/meshes/front_sonar.stl" />
 			</geometry>
 			<material name="SonarYellow">
@@ -203,5 +203,5 @@
 			<origin xyz="0 0 0" rpy="0 0 0" />
 			<geometry>
-				<mesh filename="$(find udm_pioneer_p3dx)/p3dx_description/meshes/lms100.dae" />
+				<mesh filename="package://udm_pioneer_p3dx/p3dx_description/meshes/lms100.dae" />
 			</geometry>
 		</visual>

File: install/udm_pioneer_p3dx/share/udm_pioneer_p3dx/urdf/pioneer3dx_wheel.xacro (robot description, xacro)
@@ -32,5 +32,5 @@
 				<origin xyz="0 0 0" rpy="0 0 0" />
 				<geometry name="pioneer_geom">
-					<mesh filename="package://p3dx_description/meshes/${suffix}_wheel.stl" />
+					<mesh filename="$(find udm_pioneer_p3dx)/p3dx_description/meshes/${suffix}_wheel.stl" />
 				</geometry>
 				<material name="WheelBlack">
@@ -62,5 +62,5 @@
 				<origin xyz="0 0 0" rpy="0 0 0" />
 				<geometry name="pioneer_geom">
-					<mesh filename="package://p3dx_description/meshes/${suffix}_hubcap.stl" />
+					<mesh filename="$(find udm_pioneer_p3dx)/p3dx_description/meshes/${suffix}_hubcap.stl" />
 				</geometry>
 				<material name="HubcapYellow">

Commit message: Getting left wheel to show!

File: install/udm_pioneer_p3dx/share/udm_pioneer_p3dx/urdf/pioneer3dx.xacro (robot description, xacro)
@@ -13,7 +13,5 @@
  -->
 <robot name="pioneer3dx" xmlns:xacro="http://ros.org/wiki/xacro">
-  <!-- import all gazebo-customization elements, including gazebo colors -->
-  <!-- <xacro:include filename="$(find udm_pioneer_p3dx)/urdf/pioneer3dx.gazebo.xacro" /> -->
-  <!-- import the pioneer 3dx's wheels -->
+<xacro:include filename="$(find udm_pioneer_p3dx)/urdf/pioneer3dx_wheel.xacro"/>
 <link name="base_cover">
    </link>
@@ -223,3 +221,65 @@
 		<child link="lms100" />
 	</joint>
+     <gazebo reference="p3dx_left_wheel">
+   	<material>Gazebo/Black</material>
+   </gazebo>
+      <gazebo reference="p3dx_left_hubcap">
+   	<material>Gazebo/Yellow</material>
+   </gazebo>
+	<!-- LEFT WHEEL -->
+		<!-- wheel -->
+	<link name="p3dx_left_wheel">
+		<inertial>
+			<mass value="0.5" />
+			<origin xyz="0 0 0" />
+			<inertia ixx="0.012411765597" ixy="0" ixz="0" iyy="0.015218160428"
+				iyz="0" izz="0.011763977943" />
+		</inertial>
+		<visual>
+			<origin xyz="0 0 0" rpy="0 0 0" />
+			<geometry>
+				<mesh filename="package://udm_pioneer_p3dx/p3dx_description/meshes/left_wheel.stl" />
+			</geometry>
+		</visual>
+		<collision>
+			<origin xyz="0 0 0" rpy="-1.57079635 0 0" />
+			<geometry>
+				<cylinder radius="0.09" length="0.01" />
+			</geometry>
+		</collision>
+	</link>
+	<joint name="base_left_wheel_joint" type="continuous">
+		<axis xyz="0 1 0" />
+		<anchor xyz="0 0 0" />
+		<limit effort="100" velocity="100" />
+		<joint_properties damping="0.0" friction="0.0" />
+		<origin xyz="0 0.158 0.091" rpy="0 0 0" />
+		<parent link="base_link" />
+		<child link="p3dx_left_wheel" />
+	</joint>
+	<link name="p3dx_left_hubcap">
+		<inertial>
+			<mass value="0.01" />
+			<origin xyz="0 0 0" />
+			<inertia ixx="0.012411765597" ixy="0" ixz="0" iyy="0.015218160428"
+				iyz="0" izz="0.011763977943" />
+		</inertial>
+		<visual>
+			<origin xyz="0 0 0" rpy="0 0 0" />
+			<geometry>
+				<mesh filename="package://udm_pioneer_p3dx/p3dx_description/meshes/left_hubcap.stl" />
+			</geometry>
+		</visual>
+		<collision>
+			<origin xyz="0 0 0" rpy="0 0 0" />
+			<geometry>
+				<box size="0 0 0" />
+			</geometry>
+		</collision>
+	</link>
+	<joint name="base_left_hubcap_joint" type="fixed">
+		<origin xyz="0 0 0" rpy="0 0 0" />
+		<parent link="p3dx_left_wheel" />
+		<child link="p3dx_left_hubcap" />
+	</joint>
 </robot>

File: install/udm_pioneer_p3dx/share/udm_pioneer_p3dx/urdf/pioneer3dx_wheel.xacro (robot description, xacro)
@@ -29,17 +29,13 @@
 					iyz="0" izz="0.011763977943" />
 			</inertial>
-			<visual name="p3dx_${suffix}_wheel_vis">
+			<visual>
 				<origin xyz="0 0 0" rpy="0 0 0" />
-				<geometry name="pioneer_geom">
-					<mesh filename="$(find udm_pioneer_p3dx)/p3dx_description/meshes/${suffix}_wheel.stl" />
+				<geometry>
+					<mesh filename="package://udm_pioneer_p3dx/p3dx_description/meshes/${suffix}_wheel.stl" />
 				</geometry>
-				<material name="WheelBlack">
-					<color rgba="0.117 0.117 0.117 1" />
-				</material>
 			</visual>
 			<collision>
 				<origin xyz="0 0 0" rpy="${-3.1415927/2} 0 0" />
 				<geometry>
-					<!--<mesh filename="package://p3dx_description/meshes/${suffix}_wheel.stl"/> -->
 					<cylinder radius="0.09" length="0.01" />
 				</geometry>
@@ -59,12 +55,9 @@
 					iyz="0" izz="0.011763977943" />
 			</inertial>
-			<visual name="p3dx_${suffix}_hubcap_vis">
+			<visual>
 				<origin xyz="0 0 0" rpy="0 0 0" />
-				<geometry name="pioneer_geom">
-					<mesh filename="$(find udm_pioneer_p3dx)/p3dx_description/meshes/${suffix}_hubcap.stl" />
+				<geometry>
+					<mesh filename="package://udm_pioneer_p3dx/p3dx_description/meshes/${suffix}_hubcap.stl" />
 				</geometry>
-				<material name="HubcapYellow">
-					<color rgba="1.0 0.811 0.151 1.0" />
-				</material>
 			</visual>
 			<collision>
@@ -93,14 +86,4 @@
       </actuator>
     </transmission>
-		<gazebo reference="p3dx_${suffix}_hubcap">
-			<material>Gazebo/Yellow</material>
-		</gazebo>
-		<gazebo reference="p3dx_${suffix}_wheel">
-			<material>Gazebo/Black</material>
-			<mu1>0.5</mu1>
-			<mu2>50.0</mu2>
-			<kp>100000000.0</kp>
-			<kd>1.0</kd>
-		</gazebo>
 	</xacro:macro>
 </robot>

Commit message: getting full robot to show

File: install/udm_pioneer_p3dx/share/udm_pioneer_p3dx/urdf/pioneer3dx.xacro (robot description, xacro)
@@ -283,3 +283,80 @@
 		<child link="p3dx_left_hubcap" />
 	</joint>
+    <transmission name="base_link_left_wheel_trans">
+      <type>pr2_mechanism_model/SimpleTransmission</type>
+      <joint name="base_left_wheel_joint" />
+      <actuator name="base_left_wheel_motor">
+        <hardwareInterface>VelocityJointInterface</hardwareInterface>
+        <mechanicalReduction>${624/35 * 80/19}</mechanicalReduction>
+      </actuator>
+    </transmission>
+     <gazebo reference="p3dx_right_wheel">
+   	<material>Gazebo/Black</material>
+   </gazebo>
+      <gazebo reference="p3dx_right_hubcap">
+   	<material>Gazebo/Yellow</material>
+   </gazebo>
+	<!-- RIGHT WHEEL -->
+	<link name="p3dx_right_wheel">
+		<inertial>
+			<mass value="0.5" />
+			<origin xyz="0 0 0" />
+			<inertia ixx="0.012411765597" ixy="0" ixz="0" iyy="0.015218160428"
+				iyz="0" izz="0.011763977943" />
+		</inertial>
+		<visual>
+			<origin xyz="0 0 0" rpy="0 0 0" />
+			<geometry>
+				<mesh filename="package://udm_pioneer_p3dx/p3dx_description/meshes/right_wheel.stl" />
+			</geometry>
+		</visual>
+		<collision>
+			<origin xyz="0 0 0" rpy="-1.57079635 0 0" />
+			<geometry>
+				<cylinder radius="0.09" length="0.01" />
+			</geometry>
+		</collision>
+	</link>
+	<joint name="base_right_wheel_joint" type="continuous">
+		<axis xyz="0 1 0" />
+		<anchor xyz="0 0 0" />
+		<limit effort="100" velocity="100" />
+		<joint_properties damping="0.0" friction="0.0" />
+		<origin xyz="0 -0.158 0.091" rpy="0 0 0" />
+		<parent link="base_link" />
+		<child link="p3dx_right_wheel" />
+	</joint>
+	<link name="p3dx_right_hubcap">
+		<inertial>
+			<mass value="0.01" />
+			<origin xyz="0 0 0" />
+			<inertia ixx="0.012411765597" ixy="0" ixz="0" iyy="0.015218160428"
+				iyz="0" izz="0.011763977943" />
+		</inertial>
+		<visual>
+			<origin xyz="0 0 0" rpy="0 0 0" />
+			<geometry>
+				<mesh filename="package://udm_pioneer_p3dx/p3dx_description/meshes/right_hubcap.stl" />
+			</geometry>
+		</visual>
+		<collision>
+			<origin xyz="0 0 0" rpy="0 0 0" />
+			<geometry>
+				<box size="0 0 0" />
+			</geometry>
+		</collision>
+	</link>
+	<joint name="base_right_hubcap_joint" type="fixed">
+		<origin xyz="0 0 0" rpy="0 0 0" />
+		<parent link="p3dx_right_wheel" />
+		<child link="p3dx_right_hubcap" />
+	</joint>
+    <transmission name="base_link_right_wheel_trans">
+      <type>pr2_mechanism_model/SimpleTransmission</type>
+      <joint name="base_right_wheel_joint" />
+      <actuator name="base_right_wheel_motor">
+        <hardwareInterface>VelocityJointInterface</hardwareInterface>
+        <mechanicalReduction>${-624/35 * 80/19}</mechanicalReduction>
+      </actuator>
+    </transmission>
 </robot>

File: install/udm_pioneer_p3dx/share/udm_pioneer_p3dx/urdf/pioneer3dx_wheel.xacro (robot description, xacro)
@@ -17,73 +17,65 @@
  -->
 <robot xmlns:xacro="http://ros.org/wiki/xacro">
-	<!-- properties (constants) -->
-	<xacro:property name="M_PI" value="3.14159" />
+<!-- properties (constants) -->
+<xacro:property name="M_PI" value="3.14159" />
 	<!-- right/left hubcap + wheel -->
-	<xacro:macro name="p3dx_wheel" params="suffix parent reflect">
+<xacro:macro name="p3dx_wheel" params="suffix parent reflect">
 		<!-- wheel -->
-		<link name="p3dx_${suffix}_wheel">
-			<inertial>
-				<mass value="0.5" />
-				<origin xyz="0 0 0" />
-				<inertia ixx="0.012411765597" ixy="0" ixz="0" iyy="0.015218160428"
-					iyz="0" izz="0.011763977943" />
-			</inertial>
-			<visual>
-				<origin xyz="0 0 0" rpy="0 0 0" />
-				<geometry>
-					<mesh filename="package://udm_pioneer_p3dx/p3dx_description/meshes/${suffix}_wheel.stl" />
-				</geometry>
-			</visual>
-			<collision>
-				<origin xyz="0 0 0" rpy="${-3.1415927/2} 0 0" />
-				<geometry>
-					<cylinder radius="0.09" length="0.01" />
-				</geometry>
-			</collision>
-		</link>
-		<joint name="base_${suffix}_hubcap_joint" type="fixed">
+	<link name="p3dx_${suffix}_wheel">
+		<inertial>
+			<mass value="0.5" />
+			<origin xyz="0 0 0" />
+			<inertia ixx="0.012411765597" ixy="0" ixz="0" iyy="0.015218160428"
+				iyz="0" izz="0.011763977943" />
+		</inertial>
+		<visual>
 			<origin xyz="0 0 0" rpy="0 0 0" />
-			<parent link="p3dx_${suffix}_wheel" />
-			<child link="p3dx_${suffix}_hubcap" />
-		</joint>
-		<!-- hubcap -->
-		<link name="p3dx_${suffix}_hubcap">
-			<inertial>
-				<mass value="0.01" />
-				<origin xyz="0 0 0" />
-				<inertia ixx="0.012411765597" ixy="0" ixz="0" iyy="0.015218160428"
-					iyz="0" izz="0.011763977943" />
-			</inertial>
-			<visual>
-				<origin xyz="0 0 0" rpy="0 0 0" />
-				<geometry>
-					<mesh filename="package://udm_pioneer_p3dx/p3dx_description/meshes/${suffix}_hubcap.stl" />
-				</geometry>
-			</visual>
-			<collision>
-				<origin xyz="0 0 0" rpy="0 0 0" />
-				<geometry>
-					<box size="0 0 0" />
-				</geometry>
-			</collision>
-		</link>
-		<joint name="base_${suffix}_wheel_joint" type="continuous">
-			<axis xyz="0 1 0" />
-			<anchor xyz="0 0 0" />
-			<limit effort="100" velocity="100" />
-			<joint_properties damping="0.0" friction="0.0" />
-			<origin xyz="0 ${reflect*0.158} 0.091" rpy="0 0 0" />
-			<parent link="base_link" />
-			<child link="p3dx_${suffix}_wheel" />
-		</joint>
-		<!-- gazebo elements -->
-    <transmission name="${parent}_${suffix}_wheel_trans">
-      <type>pr2_mechanism_model/SimpleTransmission</type>
-      <joint name="base_${suffix}_wheel_joint" />
-      <actuator name="base_${suffix}_wheel_motor">
-        <hardwareInterface>VelocityJointInterface</hardwareInterface>
-        <mechanicalReduction>${reflect * 624/35 * 80/19}</mechanicalReduction>
-      </actuator>
-    </transmission>
-	</xacro:macro>
+			<geometry>
+				<mesh filename="package://udm_pioneer_p3dx/p3dx_description/meshes/${suffix}_wheel.stl" />
+			</geometry>
+		</visual>
+		<collision>
+			<origin xyz="0 0 0" rpy="${-3.1415927/2} 0 0" />
+			<geometry>
+				<cylinder radius="0.09" length="0.01" />
+			</geometry>
+		</collision>
+	</link>
+	<joint name="base_${suffix}_wheel_joint" type="continuous">
+		<axis xyz="0 1 0" />
+		<anchor xyz="0 0 0" />
+		<limit effort="100" velocity="100" />
+		<joint_properties damping="0.0" friction="0.0" />
+		<origin xyz="0 ${reflect*0.158} 0.091" rpy="0 0 0" />
+		<parent link="base_link" />
+		<child link="p3dx_${suffix}_wheel" />
+	</joint>
+	<!-- hubcap -->
+	<link name="p3dx_${suffix}_hubcap">
+		<inertial>
+			<mass value="0.01" />
+			<origin xyz="0 0 0" />
+			<inertia ixx="0.012411765597" ixy="0" ixz="0" iyy="0.015218160428"
+				iyz="0" izz="0.011763977943" />
+		</inertial>
+		<visual>
+			<origin xyz="0 0 0" rpy="0 0 0" />
+			<geometry>
+				<mesh filename="package://udm_pioneer_p3dx/p3dx_description/meshes/${suffix}_hubcap.stl" />
+			</geometry>
+		</visual>
+		<collision>
+			<origin xyz="0 0 0" rpy="0 0 0" />
+			<geometry>
+				<box size="0 0 0" />
+			</geometry>
+		</collision>
+	</link>
+	<joint name="base_${suffix}_hubcap_joint" type="fixed">
+		<origin xyz="0 0 0" rpy="0 0 0" />
+		<parent link="p3dx_${suffix}_wheel" />
+		<child link="p3dx_${suffix}_hubcap" />
+	</joint>
+	<!-- gazebo elements -->
+</xacro:macro>
 </robot>
