Commit message: Updating plugin

File: install/udm_pioneer_p3dx/share/udm_pioneer_p3dx/urdf/pioneer3dx.xacro (robot description, xacro)
@@ -14,6 +14,18 @@
 <robot name="pioneer3dx" xmlns:xacro="http://ros.org/wiki/xacro">
 <xacro:include filename="$(find udm_pioneer_p3dx)/urdf/pioneer3dx_wheel.xacro"/>
-<link name="base_cover">
-   </link>
+  <!-- ground truth -->
+	<gazebo>
+		<plugin name="p3d_base_controller" filename="libgazebo_ros_p3d.so">
+			<always_on>true</always_on>
+			<update_rate>100.0</update_rate>
+			<body_name>base_link</body_name>
+			<topic_name>base_pose_ground_truth</topic_name>
+			<gaussian_noise>0.01</gaussian_noise>
+			<frame_name>map</frame_name>
+			<!-- initialize odometry for fake localization -->
+			<xyz_offset>0 0 0</xyz_offset>
+			<rpy_offset>0 0 0</rpy_offset>
+		</plugin>
+	</gazebo>
     <gazebo reference="base_link">
    	<material>Gazebo/RedBright</material>
@@ -40,8 +52,8 @@
 		</collision>
 	</link>
-   <joint name="base_cover_joint" type="fixed">
-     <parent link="base_cover"/>
-     <child link="base_link"/>
-   </joint>
+   <!-- <joint name="base_link_joint" type="fixed"> -->
+   <!--    <parent link="base_cover"/> -->
+  <!--     <child link="base_link"/> -->
+  <!--   </joint> -->
  <gazebo reference="top_plate">
    	<material>Gazebo/Black</material>
@@ -287,6 +299,6 @@
       <joint name="base_left_wheel_joint" />
       <actuator name="base_left_wheel_motor">
-        <hardwareInterface>VelocityJointInterface</hardwareInterface>
-        <mechanicalReduction>${624/35 * 80/19}</mechanicalReduction>
+        <hardware_interface>VelocityJointInterface</hardware_interface>
+        <mechanical_reduction>${624/35 * 80/19}</mechanical_reduction>
       </actuator>
     </transmission>
@@ -356,7 +368,63 @@
       <joint name="base_right_wheel_joint" />
       <actuator name="base_right_wheel_motor">
-        <hardwareInterface>VelocityJointInterface</hardwareInterface>
-        <mechanicalReduction>${-624/35 * 80/19}</mechanicalReduction>
+        <hardware_interface>VelocityJointInterface</hardware_interface>
+        <mechanical_reduction>${-624/35 * 80/19}</mechanical_reduction>
       </actuator>
     </transmission>
+  <!-- differential drive -->
+  <gazebo>
+    <plugin name="differential_drive_controller" filename="libgazebo_ros_diff_drive.so">
+        <always_on>true</always_on>
+        <update_rate>40</update_rate>
+        <legacy_mode>false</legacy_mode>
+        <left_joint>base_right_wheel_joint</left_joint>
+        <right_joint>base_left_wheel_joint</right_joint>
+        <wheel_separation>0.39</wheel_separation>
+        <wheel_diameter>0.15</wheel_diameter>
+        <torque>5</torque>
+        <command_topic>cmd_vel</command_topic>
+        <odometry_topic>odom</odometry_topic>
+        <odometry_frame>odom</odometry_frame>
+        <robot_base_frame>base_link</robot_base_frame>
+        <publish_wheel_tf>false</publish_wheel_tf>
+        <publish_wheel_joint_state>false</publish_wheel_joint_state>
+        <ros_debug_level>na</ros_debug_level>
+        <wheel_acceleration>0</wheel_acceleration>
+        <wheel_torque>5</wheel_torque>
+        <odometry_source>1</odometry_source>
+        <publish_tf>1</publish_tf>
+    </plugin>
+</gazebo>
+	<gazebo reference="lms100">
+	<material>Gazebo/Red</material>
+	<sensor type="ray" name="head_hokuyo_sensor">
+	<pose>0 0 0 0 0 0</pose>
+	<visualize>false</visualize>
+		<update_rate>100</update_rate>
+		<ray>
+		<scan>
+			<horizontal>
+				<samples>360</samples>
+				<resolution>1</resolution>
+				<min_angle>-1.570796</min_angle>
+				<max_angle>1.570796</max_angle>
+					</horizontal>
+				</scan>
+				<range>
+				<min>0.10</min>
+				<max>30.0</max>
+				<resolution>0.01</resolution>
+				</range>
+				<noise>
+				<type>gaussian</type>
+				<mean>0.0</mean>
+				<stddev>0.01</stddev>
+				</noise>
+		</ray>
+		<plugin name="gazebo_ros_head_hokuyo_controller" filename="libgazebo_ros_laser.so">
+			<topicName>scan</topicName>
+			<frameName>lms100</frameName>
+		</plugin>
+	</sensor>
+	</gazebo>
 </robot>

File: src/udm_pioneer_p3dx/urdf/pioneer3dx.xacro (robot description, xacro)
@@ -14,6 +14,18 @@
 <robot name="pioneer3dx" xmlns:xacro="http://ros.org/wiki/xacro">
 <xacro:include filename="$(find udm_pioneer_p3dx)/urdf/pioneer3dx_wheel.xacro"/>
-<link name="base_cover">
-   </link>
+  <!-- ground truth -->
+	<gazebo>
+		<plugin name="p3d_base_controller" filename="libgazebo_ros_p3d.so">
+			<always_on>true</always_on>
+			<update_rate>100.0</update_rate>
+			<body_name>base_link</body_name>
+			<topic_name>base_pose_ground_truth</topic_name>
+			<gaussian_noise>0.01</gaussian_noise>
+			<frame_name>map</frame_name>
+			<!-- initialize odometry for fake localization -->
+			<xyz_offset>0 0 0</xyz_offset>
+			<rpy_offset>0 0 0</rpy_offset>
+		</plugin>
+	</gazebo>
     <gazebo reference="base_link">
    	<material>Gazebo/RedBright</material>
@@ -40,8 +52,8 @@
 		</collision>
 	</link>
-   <joint name="base_cover_joint" type="fixed">
-     <parent link="base_cover"/>
-     <child link="base_link"/>
-   </joint>
+   <!-- <joint name="base_link_joint" type="fixed"> -->
+   <!--    <parent link="base_cover"/> -->
+  <!--     <child link="base_link"/> -->
+  <!--   </joint> -->
  <gazebo reference="top_plate">
    	<material>Gazebo/Black</material>
@@ -287,6 +299,6 @@
       <joint name="base_left_wheel_joint" />
       <actuator name="base_left_wheel_motor">
-        <hardwareInterface>VelocityJointInterface</hardwareInterface>
-        <mechanicalReduction>${624/35 * 80/19}</mechanicalReduction>
+        <hardware_interface>VelocityJointInterface</hardware_interface>
+        <mechanical_reduction>${624/35 * 80/19}</mechanical_reduction>
       </actuator>
     </transmission>
@@ -356,7 +368,31 @@
       <joint name="base_right_wheel_joint" />
       <actuator name="base_right_wheel_motor">
-        <hardwareInterface>VelocityJointInterface</hardwareInterface>
-        <mechanicalReduction>${-624/35 * 80/19}</mechanicalReduction>
+        <hardware_interface>VelocityJointInterface</hardware_interface>
+        <mechanical_reduction>${-624/35 * 80/19}</mechanical_reduction>
       </actuator>
     </transmission>
+  <!-- differential drive -->
+  <gazebo>
+    <plugin name="differential_drive_controller" filename="libgazebo_ros_diff_drive.so">
+        <always_on>true</always_on>
+        <update_rate>40</update_rate>
+        <legacy_mode>false</legacy_mode>
+        <left_joint>base_right_wheel_joint</left_joint>
+        <right_joint>base_left_wheel_joint</right_joint>
+        <wheel_separation>0.39</wheel_separation>
+        <wheel_diameter>0.15</wheel_diameter>
+        <torque>5</torque>
+        <command_topic>cmd_vel</command_topic>
+        <odometry_topic>odom</odometry_topic>
+        <odometry_frame>odom</odometry_frame>
+        <robot_base_frame>base_link</robot_base_frame>
+        <publish_wheel_tf>false</publish_wheel_tf>
+        <publish_wheel_joint_state>false</publish_wheel_joint_state>
+        <ros_debug_level>na</ros_debug_level>
+        <wheel_acceleration>0</wheel_acceleration>
+        <wheel_torque>5</wheel_torque>
+        <odometry_source>1</odometry_source>
+        <publish_tf>1</publish_tf>
+    </plugin>
+</gazebo>
 </robot>

Commit message: Working on fixing center wheel

File: install/udm_pioneer_p3dx/share/udm_pioneer_p3dx/urdf/pioneer3dx.xacro (robot description, xacro)
@@ -142,9 +142,9 @@
 	</link>
 	<joint name="swivel_hubcap_joint" type="continuous">
-		<origin xyz="-0.026 0 -0.016" rpy="0 0 0" />
 		<axis xyz="0 1 0" />
 		<anchor xyz="0 0 0" />
 		<limit effort="100" velocity="100" k_velocity="0" />
 		<joint_properties damping="0.0" friction="0.0" />
+		<origin xyz="-0.026 0 -0.016" rpy="0 0 0" />
 		<parent link="swivel" />
 		<child link="center_wheel" />
@@ -168,5 +168,5 @@
 		</visual>
 		<collision>
-			<origin xyz="0 0 0" rpy="${-3.1415927/2.0} 0 0" />
+			<origin xyz="0 0 0" rpy="${-pi/2.0} 0 0" />
 			<geometry>
 				<cylinder radius="0.0375" length="0.01" />
@@ -396,35 +396,3 @@
     </plugin>
 </gazebo>
-	<gazebo reference="lms100">
-	<material>Gazebo/Red</material>
-	<sensor type="ray" name="head_hokuyo_sensor">
-	<pose>0 0 0 0 0 0</pose>
-	<visualize>false</visualize>
-		<update_rate>100</update_rate>
-		<ray>
-		<scan>
-			<horizontal>
-				<samples>360</samples>
-				<resolution>1</resolution>
-				<min_angle>-1.570796</min_angle>
-				<max_angle>1.570796</max_angle>
-					</horizontal>
-				</scan>
-				<range>
-				<min>0.10</min>
-				<max>30.0</max>
-				<resolution>0.01</resolution>
-				</range>
-				<noise>
-				<type>gaussian</type>
-				<mean>0.0</mean>
-				<stddev>0.01</stddev>
-				</noise>
-		</ray>
-		<plugin name="gazebo_ros_head_hokuyo_controller" filename="libgazebo_ros_laser.so">
-			<topicName>scan</topicName>
-			<frameName>lms100</frameName>
-		</plugin>
-	</sensor>
-	</gazebo>
 </robot>

File: src/udm_pioneer_p3dx/urdf/pioneer3dx.xacro (robot description, xacro)
@@ -142,9 +142,9 @@
 	</link>
 	<joint name="swivel_hubcap_joint" type="continuous">
-		<origin xyz="-0.026 0 -0.016" rpy="0 0 0" />
 		<axis xyz="0 1 0" />
 		<anchor xyz="0 0 0" />
 		<limit effort="100" velocity="100" k_velocity="0" />
 		<joint_properties damping="0.0" friction="0.0" />
+		<origin xyz="-0.026 0 -0.016" rpy="0 0 0" />
 		<parent link="swivel" />
 		<child link="center_wheel" />
@@ -168,5 +168,5 @@
 		</visual>
 		<collision>
-			<origin xyz="0 0 0" rpy="${-3.1415927/2.0} 0 0" />
+			<origin xyz="0 0 0" rpy="${-pi/2.0} 0 0" />
 			<geometry>
 				<cylinder radius="0.0375" length="0.01" />

Commit message: Working on collisions

File: install/udm_pioneer_p3dx/share/udm_pioneer_p3dx/urdf/pioneer3dx.xacro (robot description, xacro)
@@ -32,4 +32,6 @@
    </gazebo>
   <!-- chassis -->
+  <!-- <link name="dummy_link"> -->
+  <!-- </link> -->
 	<link name="base_link">
 		<inertial>
@@ -52,8 +54,8 @@
 		</collision>
 	</link>
-   <!-- <joint name="base_link_joint" type="fixed"> -->
-   <!--    <parent link="base_cover"/> -->
-  <!--     <child link="base_link"/> -->
-  <!--   </joint> -->
+    <!-- <joint name="base_link_joint" type="fixed"> -->
+       <!-- <parent link="dummy_link"/>  -->
+       <!-- <child link="base_link"/>  -->
+     <!-- </joint>  -->
  <gazebo reference="top_plate">
    	<material>Gazebo/Black</material>
@@ -102,7 +104,7 @@
 		</visual>
 		<collision>
-			<origin xyz="0 0 0" rpy="0 0 0" />
-			<geometry>
-				<box size="0 0 0" />
+			<origin xyz="0.0 0.0 0.0" rpy="0.0 0.0 0.0" />
+			<geometry>
+				<box size="0.1 0.1 0.1" />
 			</geometry>
 		</collision>
@@ -124,10 +126,10 @@
 		<inertial>
 			<mass value="0.01" />
-			<origin xyz="0 0 0" />
+			<origin xyz="0.0 0.0 0.0" />
 			<inertia ixx="0.012411765597" ixy="-0.000711733678" ixz="0.00050272983"
 				iyy="0.015218160428" iyz="-0.000004273467" izz="0.011763977943" />
 		</inertial>
 		<visual>
-			<origin xyz="0 0 0" rpy="0 0 0" />
+			<origin xyz="0.0 0.0 0.0" rpy="0.0 0.0 0.0" />
 			<geometry>
 				<mesh filename="package://udm_pioneer_p3dx/p3dx_description/meshes/center_hubcap.stl" />
@@ -135,7 +137,7 @@
 		</visual>
 		<collision>
-			<origin xyz="0 0 0" rpy="0 0 0" />
-			<geometry>
-				<box size="0 0 0" />
+			<origin xyz="0.0 0.0 0.0" rpy="0.0 0.0 0.0" />
+			<geometry>
+				<box size="0.1 0.1 0.1" />
 			</geometry>
 		</collision>
@@ -152,4 +154,5 @@
 	 <gazebo reference="center_wheel">
    	<material>Gazebo/Black</material>
+	<self_collide>true</self_collide>
    </gazebo>
   <!-- center_wheel -->
@@ -157,10 +160,10 @@
 		<inertial>
 			<mass value="0.1" />
-			<origin xyz="0 0 0" />
+			<origin xyz="0.0 0.0 0.0" />
 			<inertia ixx="0.012411765597" ixy="-0.000711733678" ixz="0.00050272983"
 				iyy="0.015218160428" iyz="-0.000004273467" izz="0.011763977943" />
 		</inertial>
 		<visual>
-			<origin xyz="0 0 0" rpy="0 0 0" />
+			<origin xyz="0.0 0.0 0.0" rpy="0.0 0.0 0.0" />
 			<geometry>
 				<mesh filename="package://udm_pioneer_p3dx/p3dx_description/meshes/center_wheel.stl" />
@@ -168,12 +171,12 @@
 		</visual>
 		<collision>
-			<origin xyz="0 0 0" rpy="${-pi/2.0} 0 0" />
-			<geometry>
-				<cylinder radius="0.0375" length="0.01" />
-			</geometry>
+		    <origin xyz="0 0 0" rpy="${-3.1415927/2.0} 0 0"/>
+		    <geometry>
+			<cylinder radius="0.0375" length="0.01" />
+		    </geometry>
 		</collision>
 	</link>
 	<joint name="center_wheel_joint" type="fixed">
-		<origin xyz="-0.0035 0 -0.001" rpy="0 0 0"/>
+		<origin xyz="-0.0035 0.0 -0.001" rpy="0.0 0.0 0.0"/>
 		<parent link="center_wheel"/>
 		<child link="center_hubcap"/>
@@ -235,4 +238,8 @@
      <gazebo reference="p3dx_left_wheel">
    	<material>Gazebo/Black</material>
+	<mu1>0.5</mu1>
+			<mu2>50.0</mu2>
+			<kp>100000000.0</kp>
+			<kd>1.0</kd>
    </gazebo>
       <gazebo reference="p3dx_left_hubcap">
@@ -305,4 +312,8 @@
      <gazebo reference="p3dx_right_wheel">
    	<material>Gazebo/Black</material>
+	<mu1>0.5</mu1>
+			<mu2>50.0</mu2>
+			<kp>100000000.0</kp>
+			<kd>1.0</kd>
    </gazebo>
       <gazebo reference="p3dx_right_hubcap">
@@ -355,5 +366,5 @@
 			<origin xyz="0 0 0" rpy="0 0 0" />
 			<geometry>
-				<box size="0 0 0" />
+				<box size="0.01 0.01 0.01" />
 			</geometry>
 		</collision>

File: src/udm_pioneer_p3dx/urdf/pioneer3dx.xacro (robot description, xacro)
@@ -32,4 +32,6 @@
    </gazebo>
   <!-- chassis -->
+  <!-- <link name="dummy_link"> -->
+  <!-- </link> -->
 	<link name="base_link">
 		<inertial>
@@ -52,8 +54,8 @@
 		</collision>
 	</link>
-   <!-- <joint name="base_link_joint" type="fixed"> -->
-   <!--    <parent link="base_cover"/> -->
-  <!--     <child link="base_link"/> -->
-  <!--   </joint> -->
+    <!-- <joint name="base_link_joint" type="fixed"> -->
+       <!-- <parent link="dummy_link"/>  -->
+       <!-- <child link="base_link"/>  -->
+     <!-- </joint>  -->
  <gazebo reference="top_plate">
    	<material>Gazebo/Black</material>
@@ -102,5 +104,5 @@
 		</visual>
 		<collision>
-			<origin xyz="0 0 0" rpy="0 0 0" />
+			<origin xyz="0.0 0.0 0.0" rpy="0.0 0.0 0.0" />
 			<geometry>
 				<box size="0 0 0" />
@@ -124,10 +126,10 @@
 		<inertial>
 			<mass value="0.01" />
-			<origin xyz="0 0 0" />
+			<origin xyz="0.0 0.0 0.0" />
 			<inertia ixx="0.012411765597" ixy="-0.000711733678" ixz="0.00050272983"
 				iyy="0.015218160428" iyz="-0.000004273467" izz="0.011763977943" />
 		</inertial>
 		<visual>
-			<origin xyz="0 0 0" rpy="0 0 0" />
+			<origin xyz="0.0 0.0 0.0" rpy="0.0 0.0 0.0" />
 			<geometry>
 				<mesh filename="package://udm_pioneer_p3dx/p3dx_description/meshes/center_hubcap.stl" />
@@ -135,5 +137,5 @@
 		</visual>
 		<collision>
-			<origin xyz="0 0 0" rpy="0 0 0" />
+			<origin xyz="0.0 0.0 0.0" rpy="0.0 0.0 0.0" />
 			<geometry>
 				<box size="0 0 0" />
@@ -152,4 +154,5 @@
 	 <gazebo reference="center_wheel">
    	<material>Gazebo/Black</material>
+	<self_collide>true</self_collide>
    </gazebo>
   <!-- center_wheel -->
@@ -157,10 +160,10 @@
 		<inertial>
 			<mass value="0.1" />
-			<origin xyz="0 0 0" />
+			<origin xyz="0.0 0.0 0.0" />
 			<inertia ixx="0.012411765597" ixy="-0.000711733678" ixz="0.00050272983"
 				iyy="0.015218160428" iyz="-0.000004273467" izz="0.011763977943" />
 		</inertial>
 		<visual>
-			<origin xyz="0 0 0" rpy="0 0 0" />
+			<origin xyz="0.0 0.0 0.0" rpy="0.0 0.0 0.0" />
 			<geometry>
 				<mesh filename="package://udm_pioneer_p3dx/p3dx_description/meshes/center_wheel.stl" />
@@ -168,12 +171,12 @@
 		</visual>
 		<collision>
-			<origin xyz="0 0 0" rpy="${-pi/2.0} 0 0" />
-			<geometry>
-				<cylinder radius="0.0375" length="0.01" />
-			</geometry>
+		    <origin xyz="0 0 0" rpy="${-3.1415927/2.0} 0 0"/>
+		    <geometry>
+			<cylinder radius="0.0375" length="0.01" />
+		    </geometry>
 		</collision>
 	</link>
 	<joint name="center_wheel_joint" type="fixed">
-		<origin xyz="-0.0035 0 -0.001" rpy="0 0 0"/>
+		<origin xyz="-0.0035 0.0 -0.001" rpy="0.0 0.0 0.0"/>
 		<parent link="center_wheel"/>
 		<child link="center_hubcap"/>
@@ -223,5 +226,5 @@
 			<origin xyz="0 0 0" rpy="0 0 0" />
 			<geometry>
-				<box size="0.1 0.1 0.1" />
+				<box size="0 0 0" />
 			</geometry>
 		</collision>
@@ -235,4 +238,8 @@
      <gazebo reference="p3dx_left_wheel">
    	<material>Gazebo/Black</material>
+	<mu1>0.5</mu1>
+			<mu2>50.0</mu2>
+			<kp>100000000.0</kp>
+			<kd>1.0</kd>
    </gazebo>
       <gazebo reference="p3dx_left_hubcap">
@@ -305,4 +312,8 @@
      <gazebo reference="p3dx_right_wheel">
    	<material>Gazebo/Black</material>
+	<mu1>0.5</mu1>
+			<mu2>50.0</mu2>
+			<kp>100000000.0</kp>
+			<kd>1.0</kd>
    </gazebo>
       <gazebo reference="p3dx_right_hubcap">

Commit message: Fixed collisions

File: install/udm_pioneer_p3dx/share/udm_pioneer_p3dx/urdf/pioneer3dx.xacro (robot description, xacro)
@@ -106,5 +106,5 @@
 			<origin xyz="0.0 0.0 0.0" rpy="0.0 0.0 0.0" />
 			<geometry>
-				<box size="0.1 0.1 0.1" />
+				<box size="0 0 0" />
 			</geometry>
 		</collision>
@@ -139,5 +139,5 @@
 			<origin xyz="0.0 0.0 0.0" rpy="0.0 0.0 0.0" />
 			<geometry>
-				<box size="0.1 0.1 0.1" />
+				<box size="0 0 0" />
 			</geometry>
 		</collision>
@@ -154,5 +154,4 @@
 	 <gazebo reference="center_wheel">
    	<material>Gazebo/Black</material>
-	<self_collide>true</self_collide>
    </gazebo>
   <!-- center_wheel -->
@@ -171,7 +170,7 @@
 		</visual>
 		<collision>
-		    <origin xyz="0 0 0" rpy="${-3.1415927/2.0} 0 0"/>
+		    <origin xyz="0 0 0" rpy="-1.57079635 0 0"/>
 		    <geometry>
-			<cylinder radius="0.0375" length="0.01" />
+				<cylinder radius="0.0375" length="0.01" />
 		    </geometry>
 		</collision>
@@ -366,5 +365,5 @@
 			<origin xyz="0 0 0" rpy="0 0 0" />
 			<geometry>
-				<box size="0.01 0.01 0.01" />
+				<box size="0 0 0" />
 			</geometry>
 		</collision>

File: src/udm_pioneer_p3dx/urdf/pioneer3dx.xacro (robot description, xacro)
@@ -154,5 +154,4 @@
 	 <gazebo reference="center_wheel">
    	<material>Gazebo/Black</material>
-	<self_collide>true</self_collide>
    </gazebo>
   <!-- center_wheel -->
@@ -171,7 +170,7 @@
 		</visual>
 		<collision>
-		    <origin xyz="0 0 0" rpy="${-3.1415927/2.0} 0 0"/>
+		    <origin xyz="0 0 0" rpy="-1.57079635 0 0"/>
 		    <geometry>
-			<cylinder radius="0.0375" length="0.01" />
+				<cylinder radius="0.0375" length="0.01" />
 		    </geometry>
 		</collision>
@@ -226,5 +225,5 @@
 			<origin xyz="0 0 0" rpy="0 0 0" />
 			<geometry>
-				<box size="0 0 0" />
+				<box size="0.1 0.1 0.1" />
 			</geometry>
 		</collision>

Commit message: setting up movebase

File: install/udm_pioneer_p3dx/share/udm_pioneer_p3dx/urdf/pioneer3dx.xacro (robot description, xacro)
@@ -152,6 +152,6 @@
 		<child link="center_wheel" />
 	</joint>
-	 <gazebo reference="center_wheel">
-   	<material>Gazebo/Black</material>
+	<gazebo reference="center_wheel">
+   		<material>Gazebo/Black</material>
    </gazebo>
   <!-- center_wheel -->
@@ -235,10 +235,10 @@
 		<child link="lms100" />
 	</joint>
-     <gazebo reference="p3dx_left_wheel">
-   	<material>Gazebo/Black</material>
-	<mu1>0.5</mu1>
-			<mu2>50.0</mu2>
-			<kp>100000000.0</kp>
-			<kd>1.0</kd>
+    <gazebo reference="p3dx_left_wheel">
+ 	  	<material>Gazebo/Black</material>
+		<mu1>0.5</mu1>
+		<mu2>50.0</mu2>
+		<kp>100000000.0</kp>
+		<kd>1.0</kd>
    </gazebo>
       <gazebo reference="p3dx_left_hubcap">
