Commit message: Added use_sim_time, getting error with rviz

File: src/udm_pioneer_p3dx/urdf/pioneer3dx.xacro (robot description, xacro)
@@ -19,5 +19,5 @@
 			<always_on>true</always_on>
 			<update_rate>100.0</update_rate>
-			<body_name>base_link</body_name>
+			<body_name>base_footprint</body_name>
 			<topic_name>base_pose_ground_truth</topic_name>
 			<gaussian_noise>0.01</gaussian_noise>
@@ -31,4 +31,11 @@
    	<material>Gazebo/RedBright</material>
    </gazebo>
+   <!-- Base footprint -->
+   <link name="base_footprint"/>
+	<joint name="base_joint" type="fixed">
+    	<parent link="base_footprint"/>
+    	<child link="base_link" />
+    	<origin xyz="0.0 0.0 0.1" rpy="0 0 0"/>
+  	</joint>
   <!-- chassis -->
   <!-- <link name="dummy_link"> -->
@@ -431,5 +438,5 @@
         <odometry_topic>odom</odometry_topic>
         <odometry_frame>odom</odometry_frame>
-        <robot_base_frame>base_link</robot_base_frame>
+        <robot_base_frame>base_footprint</robot_base_frame>
         <publish_wheel_tf>false</publish_wheel_tf>
         <publish_wheel_joint_state>false</publish_wheel_joint_state>
