Commit message: Working SLAM map

File: src/udm_pioneer_p3dx_mappings/pioneer_p3dx_description/urdf/pioneer3dx.xacro (robot description, xacro)
@@ -6,6 +6,9 @@
   <xacro:include filename="pioneer3dx_wheel.xacro" />
   <xacro:include filename="pioneer3dx_lidar.xacro" />
+<!-- base link-->
+ <link name="base_link">
+    </link>
   <!-- chassis -->
-	<link name="base_link">
+	<link name="chassis">
 		<inertial>
 			<mass value="3.5" />
@@ -30,4 +33,18 @@
 		</collision>
 	</link>
+    <joint name="chassis_joint" type="fixed">
+        <parent link="base_link"/>
+        <child link="chassis"/>
+        <origin xyz="-0.05 0 0" />
+    </joint>
+	   <!-- BASE_FOOTPRINT LINK -->
+    <joint name="base_footprint_joint" type="fixed">
+        <parent link="base_link"/>
+        <child link="base_footprint"/>
+        <origin xyz="0 0 0" rpy="0 0 0"/>
+    </joint>
+	 <link name="base_footprint">
+    </link>
+	<!-- Just added base footprint-->
   <!-- top_plate -->
 	<link name="top_plate">
@@ -55,5 +72,5 @@
 	<joint name="base_top_joint" type="fixed">
 		<origin xyz="-0.045 0 0.234" rpy="0 0 0" />
-		<parent link="base_link" />
+		<parent link="chassis" />
 		<child link="top_plate" />
 	</joint>
@@ -87,5 +104,5 @@
 		<limit effort="100" velocity="100" k_velocity="0" />
 		<joint_properties damping="0.0" friction="0.0" />
-		<parent link="base_link" />
+		<parent link="chassis" />
 		<child link="swivel" />
 	</joint>
@@ -152,6 +169,6 @@
 		<child link="center_hubcap"/>
 	</joint>
-	<xacro:p3dx_wheel suffix="left" parent="base_link" reflect="1"/>
-	<xacro:p3dx_wheel suffix="right" parent="base_link" reflect="-1"/>
+	<xacro:p3dx_wheel suffix="left" parent="chassis" reflect="1"/>
+	<xacro:p3dx_wheel suffix="right" parent="chassis" reflect="-1"/>
   <!-- front_sonar -->
 	<link name="front_sonar">
@@ -179,5 +196,5 @@
 	<joint name="base_front_joint" type="fixed">
 		<origin rpy="0 0 0" xyz="0.109 0 0.209" />
-		<parent link="base_link" />
+		<parent link="chassis" />
 		<child link="front_sonar" />
 	</joint>
