Commit message: Making robot model show with rviz2

File: src/udm_pioneer_p3dx_mappings/pioneer_p3dx_description/urdf/pioneer3dx.gazebo.xacro (robot description, xacro)
@@ -4,9 +4,9 @@
   <xacro:property name="ns" value="p3dx" />
   <!-- ros_control plugin -->
-  <gazebo>
+  <!-- <gazebo>
     <plugin name="gazebo_ros_control" filename="libgazebo_ros_control.so">
       <robotNamespace>/${ns}</robotNamespace>
     </plugin>
-  </gazebo>
+  </gazebo> -->
   <!-- base_link -->
 	<gazebo reference="base_link">
@@ -40,15 +40,23 @@
 	<gazebo>
 		<plugin name="differential_drive_controller" filename="libgazebo_ros_diff_drive.so">
-			<alwaysOn>true</alwaysOn>
-			<updateRate>100</updateRate>
-			<leftJoint>base_right_wheel_joint</leftJoint>
-			<rightJoint>base_left_wheel_joint</rightJoint>
-			<wheelSeparation>0.39</wheelSeparation>
-			<wheelDiameter>0.15</wheelDiameter>
+		  	<always_on>true</always_on>
+			<update_rate>40</update_rate>
+			<legacy_mode>false</legacy_mode>
+			<left_joint>base_right_wheel_joint</left_joint>
+			<right_joint>base_left_wheel_joint</right_joint>
+			<wheel_separation>0.39</wheel_separation>
+			<wheel_diameter>0.15</wheel_diameter>
 			<torque>5</torque>
-			<commandTopic>${ns}/cmd_vel</commandTopic>
-			<odometryTopic>${ns}/odom</odometryTopic>
-			<odometryFrame>odom</odometryFrame>
-			<robotBaseFrame>base_link</robotBaseFrame>
+			<command_topic>cmd_vel</command_topic>
+			<odometry_topic>odom</odometry_topic>
+			<odometry_frame>odom</odometry_frame>
+			<robot_base_frame>base_link</robot_base_frame>
+			<publish_wheel_tf>false</publish_wheel_tf>
+			<publish_wheel_joint_state>false</publish_wheel_joint_state>
+			<ros_debug_level>na</ros_debug_level>
+			<wheel_acceleration>0</wheel_acceleration>
+			<wheel_torque>5</wheel_torque>
+			<odometry_source>1</odometry_source>
+			<publish_tf>1</publish_tf>
 		</plugin>
 	</gazebo>
@@ -56,13 +64,13 @@
 	<gazebo>
 		<plugin name="p3d_base_controller" filename="libgazebo_ros_p3d.so">
-			<alwaysOn>true</alwaysOn>
-			<updateRate>100.0</updateRate>
-			<bodyName>base_link</bodyName>
-			<topicName>${ns}/base_pose_ground_truth</topicName>
-			<gaussianNoise>0.01</gaussianNoise>
-			<frameName>map</frameName>
+			<always_on>true</always_on>
+			<update_rate>100.0</update_rate>
+			<body_name>base_link</body_name>
+			<topic_name>${ns}/base_pose_ground_truth</topic_name>
+			<gaussian_noise>0.01</gaussian_noise>
+			<frame_name>map</frame_name>
 			<!-- initialize odometry for fake localization -->
-			<xyzOffsets>0 0 0</xyzOffsets>
-			<rpyOffsets>0 0 0</rpyOffsets>
+			<xyz_offset>0 0 0</xyz_offset>
+			<rpy_offset>0 0 0</rpy_offset>
 		</plugin>
 	</gazebo>
@@ -94,6 +102,6 @@
 			</ray>
 			<plugin name="gazebo_ros_head_hokuyo_controller" filename="libgazebo_ros_laser.so">
-				<topicName>${ns}/laser/scan</topicName>
-				<frameName>lms100</frameName>
+				<topic_name>${ns}/laser/scan</topic_name>
+				<frame_name>lms100</frame_name>
 			</plugin>
 		</sensor>

File: src/udm_pioneer_p3dx_mappings/pioneer_p3dx_description/urdf/pioneer3dx.xacro (robot description, xacro)
@@ -16,5 +16,5 @@
 			<origin xyz="-0.045 0 0.148" rpy="0 0 0" />
 			<geometry name="pioneer_geom">
-				<mesh filename="package://p3dx_description/meshes/chassis.stl" />
+				<mesh filename="package://udm_pioneer_p3dx_mappings/pioneer_p3dx_description/meshes/chassis.stl" />
 			</geometry>
 			<material name="ChassisRed">
@@ -39,5 +39,5 @@
 			<origin xyz="0 0 0" rpy="0 0 0" />
 			<geometry name="top_geom">
-				<mesh filename="package://p3dx_description/meshes/top.stl" />
+				<mesh filename="package://udm_pioneer_p3dx_mappings/pioneer_p3dx_description/meshes/top.stl" />
 			</geometry>
 			<material name="TopBlack">
@@ -67,5 +67,5 @@
 			<origin xyz="0 0 0" rpy="0 0 0" />
 			<geometry name="pioneer_geom">
-				<mesh filename="package://p3dx_description/meshes/swivel.stl" />
+				<mesh filename="package://udm_pioneer_p3dx_mappings/pioneer_p3dx_description/meshes/swivel.stl" />
 			</geometry>
 			<material name="swivel">
@@ -100,5 +100,5 @@
 			<origin xyz="0 0 0" rpy="0 0 0" />
 			<geometry name="pioneer_geom">
-				<mesh filename="package://p3dx_description/meshes/center_hubcap.stl" />
+				<mesh filename="package://udm_pioneer_p3dx_mappings/pioneer_p3dx_description/meshes/center_hubcap.stl" />
 			</geometry>
 			<material name="swivel">
@@ -133,5 +133,5 @@
 			<origin xyz="0 0 0" rpy="0 0 0" />
 			<geometry name="pioneer_geom">
-				<mesh filename="package://p3dx_description/meshes/center_wheel.stl" />
+				<mesh filename="package://udm_pioneer_p3dx_mappings/pioneer_p3dx_description/meshes/center_wheel.stl" />
 			</geometry>
 			<material name="WheelBlack">
@@ -163,5 +163,5 @@
 			<origin rpy="0 0 0" xyz="0 0 0" />
 			<geometry name="pioneer_geom">
-				<mesh filename="package://p3dx_description/meshes/front_sonar.stl" />
+				<mesh filename="package://udm_pioneer_p3dx_mappings/pioneer_p3dx_description/meshes/front_sonar.stl" />
 			</geometry>
 			<material name="SonarYellow">
@@ -191,5 +191,5 @@
 			<origin xyz="0 0 0" rpy="0 0 0" />
 			<geometry>
-				<mesh filename="package://p3dx_description/meshes/lms100.dae" />
+				<mesh filename="package://udm_pioneer_p3dx_mappings/pioneer_p3dx_description/meshes/lms100.dae" />
 			</geometry>
 		</visual>

File: src/udm_pioneer_p3dx_mappings/pioneer_p3dx_description/urdf/pioneer3dx_wheel.xacro (robot description, xacro)
@@ -16,5 +16,5 @@
 				<origin xyz="0 0 0" rpy="0 0 0" />
 				<geometry name="pioneer_geom">
-					<mesh filename="package://p3dx_description/meshes/${suffix}_wheel.stl" />
+					<mesh filename="package://udm_pioneer_p3dx_mappings/pioneer_p3dx_description/meshes/${suffix}_wheel.stl" />
 				</geometry>
 				<material name="WheelBlack">
@@ -45,5 +45,5 @@
 				<origin xyz="0 0 0" rpy="0 0 0" />
 				<geometry name="pioneer_geom">
-					<mesh filename="package://p3dx_description/meshes/${suffix}_hubcap.stl" />
+					<mesh filename="package://udm_pioneer_p3dx_mappings/pioneer_p3dx_description/meshes/${suffix}_hubcap.stl" />
 				</geometry>
 				<material name="HubcapYellow">
@@ -68,4 +68,5 @@
 		</joint>
 		<!-- gazebo elements -->
+<!--
     <transmission name="${parent}_${suffix}_wheel_trans">
       <type>pr2_mechanism_model/SimpleTransmission</type>
@@ -75,5 +76,5 @@
         <mechanicalReduction>${reflect * 624/35 * 80/19}</mechanicalReduction>
       </actuator>
-    </transmission>
+    </transmission> -->
 		<gazebo reference="p3dx_${suffix}_hubcap">
 			<material>Gazebo/Yellow</material>

Commit message: Working on robot

File: src/udm_pioneer_p3dx_mappings/pioneer_p3dx_description/urdf/pioneer3dx.gazebo.xacro (robot description, xacro)
@@ -34,7 +34,7 @@
 	</gazebo>
   <!-- front_sonar -->
-  <gazebo reference="front_sonar">
-    <material value="Gazebo/Yellow" />
-  </gazebo>
+   <gazebo reference="front_sonar">
+   	<material>Gazebo/Yellow</material>
+   </gazebo>
   <!-- differential drive -->
 	<gazebo>

File: src/udm_pioneer_p3dx_mappings/pioneer_p3dx_description/urdf/pioneer3dx.xacro (robot description, xacro)
@@ -36,5 +36,5 @@
 			<inertia ixx="1" ixy="0" ixz="0" iyy="1" iyz="0" izz="1" />
 		</inertial>
-		<visual name="base_visual">
+		<visual name="top_plate_visual">
 			<origin xyz="0 0 0" rpy="0 0 0" />
 			<geometry name="top_geom">
@@ -64,5 +64,5 @@
 			<inertia ixx="0.01" ixy="0" ixz="0" iyy="0.01" iyz="0" izz="0.01" />
 		</inertial>
-		<visual name="base_visual">
+		<visual name="swivel_visual">
 			<origin xyz="0 0 0" rpy="0 0 0" />
 			<geometry name="pioneer_geom">
@@ -97,5 +97,5 @@
 				iyy="0.015218160428" iyz="-0.000004273467" izz="0.011763977943" />
 		</inertial>
-		<visual name="base_visual">
+		<visual name="center_hubcap_visual">
 			<origin xyz="0 0 0" rpy="0 0 0" />
 			<geometry name="pioneer_geom">
@@ -130,5 +130,5 @@
 				iyy="0.015218160428" iyz="-0.000004273467" izz="0.011763977943" />
 		</inertial>
-		<visual name="base_visual">
+		<visual name="center_wheel_visual">
 			<origin xyz="0 0 0" rpy="0 0 0" />
 			<geometry name="pioneer_geom">

File: src/udm_pioneer_p3dx_mappings/pioneer_p3dx_description/urdf/pioneer3dx_wheel.xacro (robot description, xacro)
@@ -5,4 +5,14 @@
 	<!-- right/left hubcap + wheel -->
 	<xacro:macro name="p3dx_wheel" params="suffix parent reflect">
+		<gazebo reference="p3dx_${suffix}_hubcap">
+			<material>Gazebo/Yellow</material>
+		</gazebo>
+		<gazebo reference="p3dx_${suffix}_wheel">
+			<material>Gazebo/Black</material>
+			<mu1>0.5</mu1>
+			<mu2>50.0</mu2>
+			<kp>100000000.0</kp>
+			<kd>1.0</kd>
+		</gazebo>
 		<!-- wheel -->
 		<link name="p3dx_${suffix}_wheel">
@@ -42,10 +52,10 @@
 					iyz="0" izz="0.011763977943" />
 			</inertial>
-			<visual name="base_visual">
+			<visual name="p3dx_${suffix}_hubcap">
 				<origin xyz="0 0 0" rpy="0 0 0" />
-				<geometry name="pioneer_geom">
+				<geometry>
 					<mesh filename="package://udm_pioneer_p3dx_mappings/pioneer_p3dx_description/meshes/${suffix}_hubcap.stl" />
 				</geometry>
-				<material name="HubcapYellow">
+				<material>
 					<color rgba="1.0 0.811 0.151 1.0" />
 				</material>
@@ -77,14 +87,4 @@
       </actuator>
     </transmission> -->
-		<gazebo reference="p3dx_${suffix}_hubcap">
-			<material>Gazebo/Yellow</material>
-		</gazebo>
-		<gazebo reference="p3dx_${suffix}_wheel">
-			<material>Gazebo/Black</material>
-			<mu1>0.5</mu1>
-			<mu2>50.0</mu2>
-			<kp>100000000.0</kp>
-			<kd>1.0</kd>
-		</gazebo>
 	</xacro:macro>
 </robot>

Commit message: displaying lidar

File: src/udm_pioneer_p3dx_mappings/pioneer_p3dx_description/urdf/pioneer3dx.gazebo.xacro (robot description, xacro)
@@ -75,35 +75,3 @@
 		</plugin>
 	</gazebo>
-	<!-- lms100 -->
-	<gazebo reference="lms100">
-		<sensor type="ray" name="head_hokuyo_sensor">
-			<pose>0 0 0 0 0 0</pose>
-			<visualize>false</visualize>
-			<update_rate>50</update_rate>
-			<ray>
-				<scan>
-					<horizontal>
-						<samples>360</samples>
-						<resolution>1</resolution>
-						<min_angle>-1.570796</min_angle>
-						<max_angle>1.570796</max_angle>
-					</horizontal>
-				</scan>
-				<range>
-					<min>0.10</min>
-					<max>30.0</max>
-					<resolution>0.01</resolution>
-				</range>
-				<noise>
-					<type>gaussian</type>
-					<mean>0.0</mean>
-					<stddev>0.01</stddev>
-				</noise>
-			</ray>
-			<plugin name="gazebo_ros_head_hokuyo_controller" filename="libgazebo_ros_laser.so">
-				<topic_name>${ns}/laser/scan</topic_name>
-				<frame_name>lms100</frame_name>
-			</plugin>
-		</sensor>
-	</gazebo>
 </robot>

File: src/udm_pioneer_p3dx_mappings/pioneer_p3dx_description/urdf/pioneer3dx.xacro (robot description, xacro)
@@ -5,4 +5,5 @@
   <!-- import the pioneer 3dx's wheels -->
   <xacro:include filename="pioneer3dx_wheel.xacro" />
+  <xacro:include filename="pioneer3dx_lidar.xacro" />
   <!-- chassis -->
 	<link name="base_link">
@@ -13,5 +14,5 @@
 			<inertia ixx="1" ixy="0" ixz="0" iyy="1" iyz="0" izz="1" />
 		</inertial>
-		<visual name="base_visual">
+		<visual>
 			<origin xyz="-0.045 0 0.148" rpy="0 0 0" />
 			<geometry name="pioneer_geom">
@@ -24,5 +25,5 @@
 		<collision>
 			<origin xyz="-0.045 0 0.145" rpy="0 0 0" />
-			<geometry>
+			<geometry name="base_link_geom">
 				<box size="0.35 0.25 0.14" />
 			</geometry>
@@ -36,5 +37,5 @@
 			<inertia ixx="1" ixy="0" ixz="0" iyy="1" iyz="0" izz="1" />
 		</inertial>
-		<visual name="top_plate_visual">
+		<visual>
 			<origin xyz="0 0 0" rpy="0 0 0" />
 			<geometry name="top_geom">
@@ -64,5 +65,5 @@
 			<inertia ixx="0.01" ixy="0" ixz="0" iyy="0.01" iyz="0" izz="0.01" />
 		</inertial>
-		<visual name="swivel_visual">
+		<visual>
 			<origin xyz="0 0 0" rpy="0 0 0" />
 			<geometry name="pioneer_geom">
@@ -97,5 +98,5 @@
 				iyy="0.015218160428" iyz="-0.000004273467" izz="0.011763977943" />
 		</inertial>
-		<visual name="center_hubcap_visual">
+		<visual>
 			<origin xyz="0 0 0" rpy="0 0 0" />
 			<geometry name="pioneer_geom">
@@ -130,5 +131,5 @@
 				iyy="0.015218160428" iyz="-0.000004273467" izz="0.011763977943" />
 		</inertial>
-		<visual name="center_wheel_visual">
+		<visual>
 			<origin xyz="0 0 0" rpy="0 0 0" />
 			<geometry name="pioneer_geom">
@@ -160,5 +161,5 @@
 			<inertia ixx="1" ixy="0" ixz="0" iyy="1" iyz="0" izz="1" />
 		</inertial>
-		<visual name="front_sonar_vis">
+		<visual>
 			<origin rpy="0 0 0" xyz="0 0 0" />
 			<geometry name="pioneer_geom">
@@ -181,29 +182,3 @@
 		<child link="front_sonar" />
 	</joint>
-	<!-- lms100 laser -->
-	<link name="lms100">
-		<inertial>
-			<mass value="1e-5" />
-			<origin xyz="0 0 0" rpy="0 0 0" />
-			<inertia ixx="1e-6" ixy="0" ixz="0" iyy="1e-6" iyz="0" izz="1e-6" />
-		</inertial>
-		<visual>
-			<origin xyz="0 0 0" rpy="0 0 0" />
-			<geometry>
-				<mesh filename="package://udm_pioneer_p3dx_mappings/pioneer_p3dx_description/meshes/lms100.dae" />
-			</geometry>
-		</visual>
-		<collision>
-			<origin xyz="0 0 0" rpy="0 0 0" />
-			<geometry>
-				<box size="0.1 0.1 0.1" />
-			</geometry>
-		</collision>
-	</link>
-	<joint name="lms100_joint" type="fixed">
-		<axis xyz="0 1 0" />
-		<origin xyz="0.16 0 0.15" rpy="0 0 0" />
-		<parent link="base_link" />
-		<child link="lms100" />
-	</joint>
 </robot>

File: src/udm_pioneer_p3dx_mappings/pioneer_p3dx_description/urdf/pioneer3dx_wheel.xacro (robot description, xacro)
@@ -23,5 +23,5 @@
 					iyz="0" izz="0.011763977943" />
 			</inertial>
-			<visual name="base_visual">
+			<visual>
 				<origin xyz="0 0 0" rpy="0 0 0" />
 				<geometry name="pioneer_geom">
@@ -52,10 +52,10 @@
 					iyz="0" izz="0.011763977943" />
 			</inertial>
-			<visual name="p3dx_${suffix}_hubcap">
+			<visual>
 				<origin xyz="0 0 0" rpy="0 0 0" />
-				<geometry>
+				<geometry name="${suffix}_hubcap">
 					<mesh filename="package://udm_pioneer_p3dx_mappings/pioneer_p3dx_description/meshes/${suffix}_hubcap.stl" />
 				</geometry>
-				<material>
+				<material name="Test">
 					<color rgba="1.0 0.811 0.151 1.0" />
 				</material>

Commit message: Setting up controllers

File: src/udm_pioneer_p3dx_mappings/pioneer_p3dx_description/urdf/pioneer3dx.gazebo.xacro (robot description, xacro)
@@ -3,10 +3,30 @@
   <!-- properties (constants) -->
   <xacro:property name="ns" value="p3dx" />
-  <!-- ros_control plugin -->
+  <!-- <ros2_control name="GazeboSystem" type="system">
+	<hardware>
+		<plugin>gazebo_ros2_control/GazeboSystem</plugin>
+	</hardware>
+	<joint name="base_left_wheel_joint">
+		<command_interface name="velocity">
+			<param name="min">-10</param>
+			<param name="max">10</param>
+		</command_interface>
+		<state_interface name="velocity"/>
+		<state_interface name="position"/>
+	</joint>
+	<joint name="base_right_wheel_joint">
+		<command_interface name="velocity">
+			<param name="min">-10</param>
+			<param name="max">10</param>
+		</command_interface>
+		<state_interface name="velocity"/>
+		<state_interface name="position"/>
+	</joint>
+  </ros2_control> -->
   <!-- <gazebo>
-    <plugin name="gazebo_ros_control" filename="libgazebo_ros_control.so">
-      <robotNamespace>/${ns}</robotNamespace>
+    <plugin name="gazebo_ros2_control" filename="libgazebo_ros2_control.so">
+	  <parameters>$(find udm_pioneer_p3dx_mappings)/pioneer_p3dx_description/config/robot_controllers.yaml</parameters>
     </plugin>
-  </gazebo> -->
+  </gazebo>  -->
   <!-- base_link -->
 	<gazebo reference="base_link">
@@ -59,4 +79,6 @@
 			<odometry_source>1</odometry_source>
 			<publish_tf>1</publish_tf>
+			<publish_odom>true</publish_odom>
+			<publish_odom_tf>true</publish_odom_tf>
 		</plugin>
 	</gazebo>

Commit message: seeing slam with rviz

File: src/udm_pioneer_p3dx_mappings/pioneer_p3dx_description/urdf/pioneer3dx.gazebo.xacro (robot description, xacro)
@@ -60,40 +60,39 @@
 	<gazebo>
 		<plugin name="differential_drive_controller" filename="libgazebo_ros_diff_drive.so">
-		  	<always_on>true</always_on>
-			<update_rate>40</update_rate>
-			<legacy_mode>false</legacy_mode>
-			<left_joint>base_right_wheel_joint</left_joint>
-			<right_joint>base_left_wheel_joint</right_joint>
-			<wheel_separation>0.39</wheel_separation>
-			<wheel_diameter>0.15</wheel_diameter>
-			<torque>5</torque>
-			<command_topic>cmd_vel</command_topic>
-			<odometry_topic>odom</odometry_topic>
-			<odometry_frame>odom</odometry_frame>
-			<robot_base_frame>base_link</robot_base_frame>
-			<publish_wheel_tf>false</publish_wheel_tf>
-			<publish_wheel_joint_state>false</publish_wheel_joint_state>
-			<ros_debug_level>Debug</ros_debug_level>
-			<wheel_acceleration>0</wheel_acceleration>
-			<wheel_torque>5</wheel_torque>
-			<odometry_source>1</odometry_source>
-			<publish_tf>1</publish_tf>
-			<publish_odom>true</publish_odom>
-			<publish_odom_tf>true</publish_odom_tf>
+		  <always_on>true</always_on>
+        <update_rate>40</update_rate>
+        <legacy_mode>false</legacy_mode>
+        <left_joint>base_right_wheel_joint</left_joint>
+        <right_joint>base_left_wheel_joint</right_joint>
+        <wheel_separation>0.39</wheel_separation>
+        <wheel_diameter>0.15</wheel_diameter>
+        <torque>5</torque>
+        <command_topic>cmd_vel</command_topic>
+        <odometry_topic>odom</odometry_topic>
+        <odometry_frame>odom</odometry_frame>
+        <robot_base_frame>base_link</robot_base_frame>
+        <publish_wheel_tf>false</publish_wheel_tf>
+        <publish_wheel_joint_state>false</publish_wheel_joint_state>
+        <ros_debug_level>na</ros_debug_level>
+        <wheel_acceleration>0</wheel_acceleration>
+        <wheel_torque>5</wheel_torque>
+        <odometry_source>1</odometry_source>
+        <publish_tf>1</publish_tf>
+		<publish_odom>true</publish_odom>
+		<publish_odom_tf>true</publish_odom_tf>
 		</plugin>
 	</gazebo>
   <!-- ground truth -->
-	<gazebo>
+	<!-- <gazebo>
 		<plugin name="p3d_base_controller" filename="libgazebo_ros_p3d.so">
 			<always_on>true</always_on>
 			<update_rate>100.0</update_rate>
-			<body_name>base_link</body_name>
+			<body_name>base_footprint</body_name>
 			<topic_name>${ns}/base_pose_ground_truth</topic_name>
 			<gaussian_noise>0.01</gaussian_noise>
 			<frame_name>map</frame_name>
-			<!-- initialize odometry for fake localization -->
 			<xyz_offset>0 0 0</xyz_offset>
 			<rpy_offset>0 0 0</rpy_offset>
 		</plugin>
-	</gazebo>
+	</gazebo>	 -->
 </robot>

File: src/udm_pioneer_p3dx_mappings/pioneer_p3dx_description/urdf/pioneer3dx.xacro (robot description, xacro)
@@ -6,9 +6,8 @@
   <xacro:include filename="pioneer3dx_wheel.xacro" />
   <xacro:include filename="pioneer3dx_lidar.xacro" />
-<!-- base link-->
- <link name="base_link">
-    </link>
-  <!-- chassis -->
-	<link name="chassis">
+<link name="base_footprint">
+</link>
+  <!-- base link -->
+	<link name="base_link">
 		<inertial>
 			<mass value="3.5" />
@@ -33,18 +32,10 @@
 		</collision>
 	</link>
-    <joint name="chassis_joint" type="fixed">
-        <parent link="base_link"/>
-        <child link="chassis"/>
-        <origin xyz="-0.05 0 0" />
-    </joint>
 	   <!-- BASE_FOOTPRINT LINK -->
     <joint name="base_footprint_joint" type="fixed">
-        <parent link="base_link"/>
-        <child link="base_footprint"/>
+        <parent link="base_footprint"/>
+        <child link="base_link"/>
         <origin xyz="0 0 0" rpy="0 0 0"/>
     </joint>
-	 <link name="base_footprint">
-    </link>
-	<!-- Just added base footprint-->
   <!-- top_plate -->
 	<link name="top_plate">
@@ -72,5 +63,5 @@
 	<joint name="base_top_joint" type="fixed">
 		<origin xyz="-0.045 0 0.234" rpy="0 0 0" />
-		<parent link="chassis" />
+		<parent link="base_link" />
 		<child link="top_plate" />
 	</joint>
@@ -104,5 +95,5 @@
 		<limit effort="100" velocity="100" k_velocity="0" />
 		<joint_properties damping="0.0" friction="0.0" />
-		<parent link="chassis" />
+		<parent link="base_link" />
 		<child link="swivel" />
 	</joint>
@@ -169,6 +160,6 @@
 		<child link="center_hubcap"/>
 	</joint>
-	<xacro:p3dx_wheel suffix="left" parent="chassis" reflect="1"/>
-	<xacro:p3dx_wheel suffix="right" parent="chassis" reflect="-1"/>
+	<xacro:p3dx_wheel suffix="left" parent="base_link" reflect="1"/>
+	<xacro:p3dx_wheel suffix="right" parent="base_link" reflect="-1"/>
   <!-- front_sonar -->
 	<link name="front_sonar">
@@ -196,5 +187,5 @@
 	<joint name="base_front_joint" type="fixed">
 		<origin rpy="0 0 0" xyz="0.109 0 0.209" />
-		<parent link="chassis" />
+		<parent link="base_link" />
 		<child link="front_sonar" />
 	</joint>
